Commit message: Update mobile_robot.urdf.xacro

File: ros_mobile_robot/urdf/mobile_robot.urdf.xacro (robot description, xacro)
@@ -1,10 +1,10 @@
 <?xml version="1.0"?>
 <robot xmlns:xacro="http://www.ros.org/wiki/xacro" name="mobile_robot">
-  <!-- Define some properties for reuse -->
-  <xacro:property name="body_height" value="0.3"/>
-  <xacro:property name="body_width" value="0.6"/>
-  <xacro:property name="body_depth" value="1"/>
-  <xacro:property name="wheel_height" value="0.1"/>
-  <xacro:property name="wheel_radius" value="0.15"/>
+  <!-- Defining some properties for reuse -->
+  <xacro:property name="body_height" value="0.15"/>
+  <xacro:property name="body_width" value="0.3"/>
+  <xacro:property name="body_depth" value="0.4"/>
+  <xacro:property name="wheel_height" value="0.05"/>
+  <xacro:property name="wheel_radius" value="0.075"/>
   <xacro:property name="wheel_color" value="yellow"/>
   <!-- Base link -->
@@ -43,5 +43,5 @@
       <origin rpy="0 0 0" xyz="0 0 0"/>
       <geometry>
-        <box size="0.2 0.2 0.2"/>
+        <box size="0.1 0.1 0.1"/>
       </geometry>
       <material name="black">
@@ -52,5 +52,5 @@
       <origin rpy="0 0 0" xyz="0 0 0"/>
       <geometry>
-        <box size="0.2 0.2 0.2"/>
+        <box size="0.1 0.1 0.1"/>
       </geometry>
     </collision>
@@ -69,5 +69,5 @@
     <parent link="base_link"/>
     <child link="head_link"/>
-    <origin xyz="0 0 ${body_height/2 + 0.1}" rpy="0 0 0"/>
+    <origin xyz="0 0 ${body_height/2 + 0.05}" rpy="0 0 0"/>
   </joint>
   <!-- Wheel macro definition -->
@@ -106,4 +106,5 @@
       <actuator name="${name}_wheel_motor">
         <mechanicalReduction>1</mechanicalReduction>
+      <hardwareInterface>hardware_interface/VelocityJointInterface</hardwareInterface>
       </actuator>
       <joint name="${name}_wheel_joint">
@@ -114,7 +115,4 @@
     <gazebo reference="${name}_wheel_link">
       <material>Gazebo/Yellow</material>
-      <mu1>0.9</mu1>
-      <mu2>0.9</mu2>
-      <selfCollide>false</selfCollide>
     </gazebo>
   </xacro:macro>
@@ -124,9 +122,232 @@
   <xacro:wheel name="rear_left" reflect_x="-1" reflect_y="1"/>
   <xacro:wheel name="rear_right" reflect_x="-1" reflect_y="-1"/>
-  <!-- Gazebo plugin for ROS control -->
-  <gazebo>
-    <plugin name="gazebo_ros_control" filename="libgazebo_ros_control.so">
-      <robotNamespace>/mobile_robot</robotNamespace>
-    </plugin>
+  <!-- LDS-02 Link -->
+  <link name="lds_link">
+    <visual>
+      <origin xyz="0 0 0" rpy="0 0 0"/>
+      <geometry>
+        <cylinder radius="0.035" length="0.035"/>
+      </geometry>
+      <material name="dark">
+        <color rgba="0.2 0.2 0.2 1"/>
+      </material>
+    </visual>
+    <collision>
+      <origin xyz="0 0 0" rpy="0 0 0"/>
+      <geometry>
+        <cylinder radius="0.035" length="0.035"/>
+      </geometry>
+    </collision>
+    <inertial>
+      <mass value="0.114"/>
+      <origin xyz="0 0 0" rpy="0 0 0"/>
+      <inertia ixx="0.001" ixy="0.0" ixz="0.0"
+               iyy="0.001" iyz="0.0"
+               izz="0.001"/>
+    </inertial>
+  </link>
+  <!-- LDS-02 Joint -->
+  <joint name="lds_joint" type="fixed">
+    <parent link="base_link"/>
+    <child link="lds_link"/>
+  <!--  <origin xyz="${body_depth/4} 0 ${body_height/2 + 0.02}" rpy="0 0 0"/> -->
+	<origin xyz="0 0 ${body_height/2 + 0.1 + 0.01}" rpy="0 0 0"/>
+  </joint>
+  <!-- LDS-02 Gazebo Plugin -->
+  <gazebo reference="lds_link">
+    <sensor type="ray" name="lds_lfcd_sensor">
+      <pose>0 0 0 0 0 0</pose>
+      <visualize>false</visualize>
+      <update_rate>5</update_rate>
+      <ray>
+        <scan>
+          <horizontal>
+            <samples>360</samples>
+            <resolution>1</resolution>
+            <min_angle>0.0</min_angle>
+            <max_angle>6.28319</max_angle>
+          </horizontal>
+        </scan>
+        <range>
+          <min>0.120</min>
+          <max>3.5</max>
+          <resolution>0.015</resolution>
+        </range>
+        <noise>
+          <type>gaussian</type>
+          <mean>0.0</mean>
+          <stddev>0.01</stddev>
+        </noise>
+      </ray>
+      <plugin name="gazebo_ros_lds_lfcd_controller" filename="libgazebo_ros_laser.so">
+        <topicName>scan</topicName>
+        <frameName>lds_link</frameName>
+      </plugin>
+    </sensor>
   </gazebo>
+  <!-- RealSense D435i Link -->
+  <link name="d435i_link">
+    <visual>
+      <origin xyz="0 0 0" rpy="0 0 0"/>
+      <geometry>
+        <box size="0.02 0.099 0.023"/>
+      </geometry>
+      <material name="aluminum">
+        <color rgba="0.5 0.5 0.5 1"/>
+      </material>
+    </visual>
+    <collision>
+      <origin xyz="0 0 0" rpy="0 0 0"/>
+      <geometry>
+        <box size="0.02 0.099 0.023"/>
+      </geometry>
+    </collision>
+    <inertial>
+      <mass value="0.072"/>
+      <origin xyz="0 0 0" rpy="0 0 0"/>
+      <inertia ixx="0.0001" ixy="0.0" ixz="0.0"
+               iyy="0.0001" iyz="0.0"
+               izz="0.0001"/>
+    </inertial>
+  </link>
+  <!-- RealSense D435i Joint -->
+  <joint name="d435i_joint" type="fixed">
+    <parent link="base_link"/>
+    <child link="d435i_link"/>
+    <origin xyz="${body_depth/2 - 0.01} 0 ${body_height/2 + 0.01}" rpy="0 0 0"/>
+  </joint>
+  <!-- RealSense D435i Gazebo Plugin -->
+  <gazebo reference="d435i_link">
+    <sensor type="depth" name="d435i">
+      <always_on>true</always_on>
+      <update_rate>30.0</update_rate>
+      <camera name="d435i">
+        <horizontal_fov>1.5184</horizontal_fov>
+        <image>
+          <width>848</width>
+          <height>480</height>
+          <format>B8G8R8</format>
+        </image>
+        <clip>
+          <near>0.1</near>
+          <far>10.0</far>
+        </clip>
+        <noise>
+          <type>gaussian</type>
+          <mean>0.0</mean>
+          <stddev>0.007</stddev>
+        </noise>
+      </camera>
+      <plugin name="d435i_controller" filename="libgazebo_ros_openni_kinect.so">
+        <baseline>0.095</baseline>
+        <alwaysOn>true</alwaysOn>
+        <updateRate>30.0</updateRate>
+        <cameraName>d435i</cameraName>
+        <imageTopicName>color/image_raw</imageTopicName>
+        <cameraInfoTopicName>color/camera_info</cameraInfoTopicName>
+        <depthImageTopicName>depth/image_rect_raw</depthImageTopicName>
+        <depthImageInfoTopicName>depth/camera_info</depthImageInfoTopicName>
+        <pointCloudTopicName>depth/color/points</pointCloudTopicName>
+        <frameName>d435i_link</frameName>
+        <pointCloudCutoff>0.1</pointCloudCutoff>
+        <pointCloudCutoffMax>10.0</pointCloudCutoffMax>
+        <distortionK1>0.00000001</distortionK1>
+        <distortionK2>0.00000001</distortionK2>
+        <distortionK3>0.00000001</distortionK3>
+        <distortionT1>0.00000001</distortionT1>
+        <distortionT2>0.00000001</distortionT2>
+      </plugin>
+    </sensor>
+    <!-- IMU sensor for D435i -->
+    <sensor name="d435i_imu" type="imu">
+      <always_on>true</always_on>
+      <update_rate>200</update_rate>
+      <visualize>true</visualize>
+      <imu>
+        <angular_velocity>
+          <x><noise type="gaussian"><mean>0.0</mean><stddev>0.00</stddev><bias_mean>0.0</bias_mean><bias_stddev>0.0</bias_stddev></noise></x>
+          <y><noise type="gaussian"><mean>0.0</mean><stddev>0.00</stddev><bias_mean>0.0</bias_mean><bias_stddev>0.0</bias_stddev></noise></y>
+          <z><noise type="gaussian"><mean>0.0</mean><stddev>0.00</stddev><bias_mean>0.0</bias_mean><bias_stddev>0.0</bias_stddev></noise></z>
+        </angular_velocity>
+        <linear_acceleration>
+          <x><noise type="gaussian"><mean>0.0</mean><stddev>0.00</stddev><bias_mean>0.0</bias_mean><bias_stddev>0.0</bias_stddev></noise></x>
+          <y><noise type="gaussian"><mean>0.0</mean><stddev>0.00</stddev><bias_mean>0.0</bias_mean><bias_stddev>0.0</bias_stddev></noise></y>
+          <z><noise type="gaussian"><mean>0.0</mean><stddev>0.00</stddev><bias_mean>0.0</bias_mean><bias_stddev>0.0</bias_stddev></noise></z>
+        </linear_acceleration>
+      </imu>
+      <plugin name="d435i_imu_controller" filename="libgazebo_ros_imu_sensor.so">
+        <topicName>d435i/imu</topicName>
+        <bodyName>d435i_link</bodyName>
+        <updateRateHZ>200.0</updateRateHZ>
+        <gaussianNoise>0.0</gaussianNoise>
+        <xyzOffset>0 0 0</xyzOffset>
+        <rpyOffset>0 0 0</rpyOffset>
+        <frameName>d435i_link</frameName>
+      </plugin>
+    </sensor>
+  </gazebo>
+  <!-- D435i specific TF frames -->
+  <link name="d435i_depth_frame"/>
+  <joint name="d435i_depth_joint" type="fixed">
+    <parent link="d435i_link"/>
+    <child link="d435i_depth_frame"/>
+    <origin xyz="0 0 0" rpy="0 0 0"/>
+  </joint>
+  <link name="d435i_color_frame"/>
+  <joint name="d435i_color_joint" type="fixed">
+    <parent link="d435i_link"/>
+    <child link="d435i_color_frame"/>
+    <origin xyz="0 0.015 0" rpy="0 0 0"/>
+  </joint>
+<!--gazebo plugin -->
+ <gazebo>
+  <plugin name="gazebo_ros_control" filename="libgazebo_ros_control.so">
+    <robotNamespace>/</robotNamespace>
+    <robotSimType>gazebo_ros_control/DefaultRobotHWSim</robotSimType>
+  </plugin>
+</gazebo>
+<!-- Front Left Wheel -->
+<transmission name="front_left_wheel_trans">
+  <type>transmission_interface/SimpleTransmission</type>
+  <joint name="front_left_wheel_joint">
+   <hardwareInterface>hardware_interface/VelocityJointInterface</hardwareInterface>
+  </joint>
+  <actuator name="front_left_wheel_motor">
+    <mechanicalReduction>1</mechanicalReduction>
+  <hardwareInterface>hardware_interface/VelocityJointInterface</hardwareInterface>
+  </actuator>
+</transmission>
+<!-- Front Right Wheel -->
+<transmission name="front_right_wheel_trans">
+  <type>transmission_interface/SimpleTransmission</type>
+  <joint name="front_right_wheel_joint">
+    <hardwareInterface>hardware_interface/VelocityJointInterface</hardwareInterface>
+  </joint>
+  <actuator name="front_right_wheel_motor">
+    <mechanicalReduction>1</mechanicalReduction>
+   <hardwareInterface>hardware_interface/VelocityJointInterface</hardwareInterface>
+  </actuator>
+</transmission>
+<!-- Rear Left Wheel -->
+<transmission name="rear_left_wheel_trans">
+  <type>transmission_interface/SimpleTransmission</type>
+  <joint name="rear_left_wheel_joint">
+    <hardwareInterface>hardware_interface/VelocityJointInterface</hardwareInterface>
+  </joint>
+  <actuator name="rear_left_wheel_motor">
+    <mechanicalReduction>1</mechanicalReduction>
+  <hardwareInterface>hardware_interface/VelocityJointInterface</hardwareInterface>
+  </actuator>
+</transmission>
+<!-- Rear Right Wheel -->
+<transmission name="rear_right_wheel_trans">
+  <type>transmission_interface/SimpleTransmission</type>
+  <joint name="rear_right_wheel_joint">
+    <hardwareInterface>hardware_interface/VelocityJointInterface</hardwareInterface>
+  </joint>
+  <actuator name="rear_right_wheel_motor">
+    <mechanicalReduction>1</mechanicalReduction>
+  <hardwareInterface>hardware_interface/VelocityJointInterface</hardwareInterface>
+  </actuator>
+</transmission>
 </robot>
